Commit message: gengxin

File: install/mower_description/share/mower_description/urdf/mower.urdf (robot description, URDF)
Before this commit: robot mower, 19 links, 18 joints
Links:
- removed link indicator_light_1
- removed link indicator_light_2
- removed link indicator_light_3
- link base_link: geometry collision box size=0.5665 0.37 0.15; visual box size=0.48 0.015 0.025
- link bumper_link: geometry collision box size=0.1 0.3 0.05; visual box size=0.1 0.3 0.05
- link front_left_caster: geometry collision cylinder length=0.03 radius=0.045; visual cylinder length=0.03 radius=0.045
- link front_right_caster: geometry collision cylinder length=0.03 radius=0.045; visual cylinder length=0.03 radius=0.045
- link laser_link: geometry visual box size=0.1 0.1 0.05; visual box size=0.102 0.102 0.012
- link left_wheel: geometry collision cylinder length=0.05 radius=0.11; visual cylinder length=0.05 radius=0.11
- link right_wheel: geometry collision cylinder length=0.05 radius=0.11; visual cylinder length=0.05 radius=0.11
- link ultrasonic_link: geometry visual box size=0.005 0.02 0.02; visual box size=0.04 0.02 0.02
Joints:
- removed joint indicator_light_1_joint
- removed joint indicator_light_2_joint
- removed joint indicator_light_3_joint
- joint blade_joint: limit effort=50 velocity=30 -> effort=50 velocity=80; origin xyz=0 0 0.045 rpy=0 0 0 -> xyz=0 0 -0.01 rpy=0 0 0
- joint bumper_joint: origin xyz=0 0 0.05 rpy=0 0 0 -> xyz=0 0 0 rpy=0 0 0
- joint camera_joint: origin xyz=0.22 0 0.215 rpy=0 0 0 -> xyz=0.22 0 0.165 rpy=0 0 0
- joint front_left_caster_joint: origin xyz=0.15 0.18 0.09 rpy=0 0 0 -> xyz=0.180 0.0925 -0.035 rpy=0 0 0
- joint front_right_caster_joint: origin xyz=0.15 -0.18 0.09 rpy=0 0 0 -> xyz=0.180 -0.0925 -0.035 rpy=0 0 0
- joint imu_joint: origin xyz=0 0 0.125 rpy=0 0 0 -> xyz=0 0 0.075 rpy=0 0 0
- joint left_wheel_joint: origin xyz=-0.2 0.2 0.11 rpy=0 0 0 -> xyz=-0.12 0.16 0.03 rpy=0 0 0
- joint lidar_mast_joint: origin xyz=0.0 0.0 0.22 rpy=0 0 0 -> xyz=0.0 0.0 0.17 rpy=0 0 0
- joint right_wheel_joint: origin xyz=-0.2 -0.2 0.11 rpy=0 0 0 -> xyz=-0.12 -0.16 0.03 rpy=0 0 0
- joint ultrasonic_joint: origin xyz=0.27 0 0.13 rpy=0 0 0 -> xyz=0.27 0 0.08 rpy=0 0 0

Commit message: gengxin

File: install/mower_description/share/mower_description/urdf/mower.urdf (robot description, URDF)
Before this commit: robot mower, 16 links, 15 joints
Joints:
- joint blade_joint: origin xyz=0 0 -0.01 rpy=0 0 0 -> xyz=0.12 0 -0.01 rpy=0 0 0
- joint bumper_joint: origin xyz=0 0 0 rpy=0 0 0 -> xyz=0.12 0 0 rpy=0 0 0
- joint camera_joint: origin xyz=0.22 0 0.165 rpy=0 0 0 -> xyz=0.34 0 0.165 rpy=0 0 0
- joint front_left_caster_joint: origin xyz=0.180 0.0925 -0.035 rpy=0 0 0 -> xyz=0.30 0.0925 -0.035 rpy=0 0 0
- joint front_right_caster_joint: origin xyz=0.180 -0.0925 -0.035 rpy=0 0 0 -> xyz=0.30 -0.0925 -0.035 rpy=0 0 0
- joint imu_joint: origin xyz=0 0 0.075 rpy=0 0 0 -> xyz=0.12 0 0.075 rpy=0 0 0
- joint left_wheel_joint: origin xyz=-0.12 0.16 0.03 rpy=0 0 0 -> xyz=0 0.16 0.03 rpy=0 0 0
- joint lidar_mast_joint: origin xyz=0.0 0.0 0.17 rpy=0 0 0 -> xyz=0.12 0.0 0.17 rpy=0 0 0
- joint right_wheel_joint: origin xyz=-0.12 -0.16 0.03 rpy=0 0 0 -> xyz=0 -0.16 0.03 rpy=0 0 0
- joint ultrasonic_joint: origin xyz=0.27 0 0.08 rpy=0 0 0 -> xyz=0.39 0 0.08 rpy=0 0 0
